Commit message: Learned urdf modelling of robot arm

File: ros2_ws/src/arduinobot_description/urdf/arduinobot.urdf.xacro (robot description, xacro)
@@ -2,4 +2,9 @@
 <robot xmlns:xacro="http://www.ros.org/wiki/xacro" name="arduinobot"> <!-- Since we are using XACRO
     Model and not plain URDF, we need to indicate the definition of this format is located-->
+    <xacro:property name="PI" value="3.14159" /> <!-- This xacro property helps to define values into
+    variables and cane be reused as property values(it's same as setting values into variables and
+    using the variables as input data) -->
+    <xacro:property name="effort" value="30.0" />
+    <xacro:property name="velocity" value="10.0" />
     <link name="world" /> <!--This
     link doesn't belong to robot yet, but will only serve to anchor the manipulator to the world
@@ -8,9 +13,11 @@
     <link name="base_link">
         <visual>
-            <origin rpy="0 0 0" xyz="0 0 0" /> <!--  rpy defines orientation and xyz defines position
+            <origin rpy="0 0 0" xyz="0 0 0.47" /> <!--  rpy defines orientation and xyz defines
+            position
             relative to link it belongs to(here it is base link)-->
             <geometry>
                 <mesh filename="package://arduinobot_description/meshes/base-support.stl"
-                    scale="0.01 0.01 0.01" /> <!-- scale is used to reduce the file size as it may be
+                    scale="0.01 0.01 0.01" /> <!-- scale is used t1 reduce the file size as it
+                may be
                 large in all directions and also must specify origin of this mesh with respect to
                 base link(like where this mesh is located and how this mesh is oriented w.r.t base
@@ -29,3 +36,98 @@
         positioned)-->
     </joint>
+    <link name="actual_base_link">
+        <visual>
+            <origin rpy="0 0 0" xyz="0 0 0.47" />
+            <geometry>
+                <mesh filename="package://arduinobot_description/meshes/base.stl"
+                    scale="0.01 0.01 0.01" />
+            </geometry>
+        </visual>
+    </link>
+    <joint name="base_joint" type="fixed">
+        <parent link="base_link" />
+        <child link="actual_base_link" />
+        <origin rpy="0 0 0" xyz="0 0 0" />
+    </joint>
+    <link name="rotative_base_link">
+        <visual>
+            <origin rpy="0 0 0" xyz="0 0 0" />
+            <geometry>
+                <mesh filename="package://arduinobot_description/meshes/rotative_base.stl"
+                    scale="0.01 0.01 0.01" />
+            </geometry>
+        </visual>
+    </link>
+    <joint name="rotative_base_joint" type="revolute">
+        <parent link="actual_base_link" />
+        <child link="rotative_base_link" />
+        <origin rpy="0 0 0" xyz="0 0 0.46" />
+        <axis xyz="0 0 1" /> <!-- uesd  in revolute joints to specify axis of rotation in xyz
+        direction-->
+        <limit lower="-${PI/2}" upper="${PI/2}" effort="${effort}" velocity="${velocity}" /> <!--
+        specifying limits of rototion of
+        joints(lower, upper). Angles are set in radians by default. Also specify the
+        maximum effort/force and velocity(if joints use same motors, use same values for
+        velocity)-->
+    </joint>
+    <link name="servo_support_link_1">
+        <visual>
+            <origin rpy="0 0 0" xyz="0 0 0" />
+            <geometry>
+                <mesh filename="package://arduinobot_description/meshes/servo-support.stl"
+                    scale="0.01 0.01 0.01" />
+            </geometry>
+        </visual>
+    </link>
+    <joint name="servo_support_link_1_joint" type="fixed">
+        <parent link="rotative_base_link" />
+        <child link="servo_support_link_1" />
+        <origin rpy="0 0 0" xyz="0 0 0" />
+    </joint>
+    <link name="servo_support_link_2">
+        <visual>
+            <origin rpy="0 0 3.14152" xyz="0 0 0" />
+            <geometry>
+                <mesh filename="package://arduinobot_description/meshes/servo-support.stl"
+                    scale="0.01 0.01 0.01" />
+            </geometry>
+        </visual>
+    </link>
+    <joint name="servo_support_link_2_joint" type="fixed">
+        <parent link="rotative_base_link" />
+        <child link="servo_support_link_2" />
+        <origin rpy="0 0 0" xyz="0 0 0" />
+    </joint>
+    <link name="arm_1_link">
+        <visual>
+            <origin rpy="0 0 0" xyz="0 0 0" />
+            <geometry>
+                <mesh filename="package://arduinobot_description/meshes/arm_1.stl"
+                    scale="0.01 0.01 0.01" />
+            </geometry>
+        </visual>
+    </link>
+    <joint name="arm_1_joint" type="revolute">
+        <parent link="servo_support_link_1" />
+        <child link="arm_1_link" />
+        <origin rpy="0 0 0" xyz="0 0 0.34" />
+        <axis xyz="0 1 0" />
+        <limit lower="-${PI/2}" upper="${PI/2}" effort="${effort}" velocity="${velocity}" />
+    </joint>
+    <link name="arm_2_link">
+        <visual>
+            <origin rpy="0 0 3.14152" xyz="0 0 -0.95" />
+            <geometry>
+                <mesh filename="package://arduinobot_description/meshes/arm_2.stl"
+                    scale="0.01 0.01 0.01" />
+            </geometry>
+        </visual>
+    </link>
+    <joint name="arm_2_joint" type="revolute">
+        <parent link="servo_support_link_2" />
+        <child link="arm_2_link" />
+        <origin rpy="0 0 0" xyz="0 0 0" />
+        <axis xyz="0 1 0" />
+        <limit lower="-${PI/2}" upper="${PI/2}" effort="${effort}" velocity="${velocity}" />
+    </joint>
 </robot>
